Commit message: urdf update 2

File: basic134/urdf/134threedof.urdf (robot description, URDF)
Before this commit: robot 134threedof, 9 links, 8 joints
Joints:
- joint elbow: origin xyz=0 0 0.0311 rpy=0 0 0 -> xyz=0 0 0.0311 rpy=0 0 1.5708
- joint lbracket: origin xyz=0 0.02999 0.09585 rpy=1.5708 0.0 0.0 -> xyz=0 0.02999 0.09585 rpy=1.5708 -1.5708 0.0
- joint lowerarm: origin xyz=0.0 0.3785 0.00285 rpy=0 0 0 -> xyz=0.3785 0.0 0.00285 rpy=0 0 0
- joint shoulder: origin xyz=0 0 0.0451 rpy=0 0 0 -> xyz=0 0 0.0451 rpy=0 0 -1.5708

Commit message: urdf finished

File: basic134/urdf/134threedof.urdf (robot description, URDF)
Before this commit: robot 134threedof, 9 links, 8 joints
Links:
- link lowerarm: geometry visual box size=0.405 0.06 0.00570
Joints:
- joint elbow: origin xyz=0 0 0.0311 rpy=0 0 1.5708 -> xyz=0 0 0.0311 rpy=0 0 0.0
- joint upperarm: origin xyz=-0.3748 0 0.0057 rpy=0 0 1.5708 -> xyz=-0.3748 0 0.0057 rpy=0 0 3.1514

Commit message: touch table working

File: basic134/urdf/134threedof.urdf (robot description, URDF)
Before this commit: robot 134threedof, 9 links, 8 joints
Joints:
- joint upperarm: origin xyz=-0.3748 0 0.0057 rpy=0 0 3.1514 -> xyz=0.0 0.3748 0.0057 rpy=0 0 1.5708

Commit message: urdf fix for table y datum

File: basic134/urdf/134threedof.urdf (robot description, URDF)
Before this commit: robot 134threedof, 9 links, 8 joints
Joints:
- joint lowerarm: origin xyz=0.3785 0.0 0.00285 rpy=0 0 0 -> xyz=0.3685 0.0 0.00285 rpy=0 0 0
- joint placement: origin xyz=0 0 0 rpy=0 0 0 -> xyz=0 0.0394 0 rpy=0 0 0

Commit message: input table touch point implemented

File: basic134/urdf/134threedof.urdf (robot description, URDF)
Before this commit: robot 134threedof, 9 links, 8 joints
Joints:
- joint placement: origin xyz=0 0.0394 0 rpy=0 0 0 -> xyz=-0.3244 0.0394 0 rpy=0 0 0
