Commit message: just committed everything for strips and checkers
might need to clean up repo after

File: threedof/urdf/threedofexample.urdf (robot description, URDF)
Before this commit: robot 134threedof, 9 links, 8 joints
Links:
- link baseplate: geometry visual box size=0.2 0.1 0.0230
- link lowerarm: geometry visual mesh filename=package://basic134/meshes/basiclink.stl
- link upperarm: geometry visual box size=0.6 0.08 0.00570
Joints:
- joint baseplate: origin xyz=0 0 0.0125 rpy=0 0 -1.5708 -> xyz=0 0 0.0230 rpy=0 0 -1.5708
- joint elbow: origin xyz=0 0 0.0311 rpy=0 0 0.0 -> xyz=0 0 0.0311 rpy=0 0 0
- joint lbracket: origin xyz=0 0.02999 0.0953 rpy=1.5708 -1.5708 0.0 -> xyz=0 0.1 0.1 rpy=0 -1.5708 1.5708
- joint lowerarm: origin xyz=0.37 0.0 0.00285 rpy=0 0 0 -> xyz=0.5 0 0.00285 rpy=0 0 0
- joint placement: origin xyz=-0.2875 0.0394 0 rpy=0 0 0 -> xyz=0 0 0 rpy=0 0 0
- joint shoulder: origin xyz=0 0 0.0451 rpy=0 0 -1.5708 -> xyz=0 0 0.0451 rpy=0 0 0
- joint upperarm: origin xyz=0.0 0.38 0.0057 rpy=0 0 1.5708 -> xyz=0.5 0 0.0057 rpy=0 0 0
