Commit message: newest commmits

File: sixdof/urdf/fivedof.urdf (robot description, URDF)
Before this commit: robot fivedof, 13 links, 12 joints
Links:
- added link tipcamera
Joints:
- added joint tipcamera: type fixed, parent rollmotor, child tipcamera, origin xyz=-0.135 0.0 0.06 rpy=0.0 0.0 0
- joint placement: origin xyz=0.0 0.0394 0.0 rpy=0 0 0 -> xyz=0.0 0.0 0.0 rpy=0 0 3.1415

Commit message: added a bunch of todos / fixmes

File: sixdof/urdf/fivedof.urdf (robot description, URDF)
Before this commit: robot fivedof, 14 links, 13 joints
Joints:
- joint baseplate: origin xyz=0 0 0.0125 rpy=0 0 -1.5708 -> xyz=0 0 0.0124 rpy=0 0 -1.5708
- joint placement: origin xyz=0.0 0.0 0.0 rpy=0 0 3.1415 -> xyz=0.7745 0.0394 0.0 rpy=0 0 3.1415

Commit message: progress

File: sixdof/urdf/fivedof.urdf (robot description, URDF)
Before this commit: robot fivedof, 14 links, 13 joints
Joints:
- joint gripper: origin xyz=0.0 0.0 0.15821 rpy=0.0 0.0 0.0 -> xyz=0.0 0.0 0.0 rpy=0.0 0.0 0.0
- joint lbracket: origin xyz=0 0.040 0.085 rpy=1.5708 -1.5708 0.0 -> xyz=0 0.040 0.1 rpy=1.5708 -1.5708 0.0
